Commit message: added realsense2 support

File: openbase2_description/urdf/openbase2.xacro (robot description, xacro)
@@ -23,4 +23,5 @@
   <!-- IMU Frame -->
   <!-- <link name="imu_frame"/> -->
+  <link name="camera_link"/>
   <!-- Joints -->
   <joint name="base_footprint_to_base_link" type="fixed">
@@ -39,3 +40,8 @@
     <origin xyz="0.1 0 0" rpy="0 0 0"/>
   </joint> -->
+  <joint name="base_link_to_camera_link" type="fixed">
+    <parent link="base_link"/>
+    <child link="camera_link"/>
+    <origin xyz="0.32 0 0.0555" rpy="0 0 0"/>
+  </joint>
 </robot>

Commit message: added rtab and updated rviz

File: openbase2_description/urdf/openbase2.xacro (robot description, xacro)
@@ -43,5 +43,5 @@
     <parent link="base_link"/>
     <child link="camera_link"/>
-    <origin xyz="0.32 0 0.0555" rpy="0 0 0"/>
+    <origin xyz="0.32 0.02 0.0665" rpy="0 0 0"/>
   </joint>
 </robot>
